Commit message: configured mock hardware

File: rpd_robot_description/urdf/rpd_robot.urdf.xacro (robot description, xacro)
@@ -1,9 +1,15 @@
 <?xml version="1.0"?>
 <robot name="rpd_robot" xmlns:xacro="http://www.ros.org/wiki/xacro">
+  <material name="black">
+    <color rgba="0 0 0 1"/>
+  </material>
   <xacro:property name="description_pkg" value="$(find rpd_robot_description)" />
-  <xacro:include filename="${description_pkg}/urdf/materials.xacro"/>
-  <xacro:include filename="${description_pkg}/urdf/properties.xacro"/>
+  <xacro:property name="config_file" value="${description_pkg}/config/urdf_config.yaml" />
+  <xacro:property name="config" value="${xacro.load_yaml(config_file)}" />
+  <xacro:property name="links" value="${config['links']}" />
+  <xacro:property name="joints" value="${config['joints']}" />
   <xacro:include filename="${description_pkg}/urdf/rpd_robot_arm.urdf.xacro"/>
   <xacro:include filename="${description_pkg}/urdf/rpd_robot_gripper.urdf.xacro"/>
-  <!-- <xacro:include filename="$(find rpd_robot_description)/urdf/rpd_robot.ros2_control.xacro"/> -->
+  <xacro:include filename="${description_pkg}/urdf/rpd_robot_ros2_control.xacro"/>
+  <!-- <xacro:include filename="${description_pkg}/urdf/rpd_robot_gazebo.xacro"/> -->
 </robot>

File: rpd_robot_description/urdf/rpd_robot_arm.urdf.xacro (robot description, xacro)
@@ -2,46 +2,59 @@
 <robot xmlns:xacro="http://www.ros.org/wiki/xacro">
   <!-- origin and geometry macro -->
-  <xacro:macro name="origin_geometry" params="number">
-    <origin rpy="0 0 0" xyz="${link_positions[number]}" />
+  <xacro:macro name="origin_geometry" params="link">
+    <origin rpy="0 0 0" xyz="${link['xyz']}" />
     <geometry>
-      <mesh filename="file://${$description_pkg}/meshes/${link_names[number]}.stl" scale="${scale}" />
+      <mesh filename="file://${description_pkg}/meshes/${link['name']}.stl" />
     </geometry>
   </xacro:macro>
+  <!-- Inertial macro -->
+  <xacro:macro name="inertial" params="link">
+    <inertial>
+      <mass value="${link['mass']}" />
+      <origin xyz="${link['com']}" rpy="0 0 0"/>
+      <inertia ixx="${link['inertia']['ixx']}" ixy="0" ixz="0"
+               iyy="${link['inertia']['iyy']}" iyz="0"
+               izz="${link['inertia']['izz']}" />
+    </inertial>
+  </xacro:macro>
   <!-- link macro -->
-  <xacro:macro name="link" params="number color:=black">
-    <link name="${link_names[number]}">
+  <xacro:macro name="link" params="link color:=black">
+    <link name="${link['name']}">
         <visual>
-        <xacro:origin_geometry number="${number}" />
-        <material name="${color}" />
+        <xacro:origin_geometry link="${link}" />
+        <material name="${link['color']}" />
         </visual>
         <collision>
-        <xacro:origin_geometry number="${number}" />
+        <xacro:origin_geometry link="${link}" />
         </collision>
+        <!-- <xacro:inertial n="${links[n]}" /> -->
     </link>
   </xacro:macro>
  <!-- joint macro -->
-  <xacro:macro name="joint" params="number lower upper velocity axis">
-    <joint name="${joint_names[number]}" type="revolute">
-        <origin rpy="0 0 0" xyz="${joint_positions[number]}"/>
-        <limit effort="${effort}" lower="${lower}" upper="${upper}" velocity="${velocity}"/>
-        <axis xyz="${axis}" />
-        <parent link="${link_names[number]}" />
-        <child link="${link_names[number + 1]}" />
+  <xacro:macro name="joint" params="joint n">
+    <joint name="${joint['name']}" type="revolute"> <!-- can keep continuous for joint_1 -->
+        <origin rpy="0 0 0" xyz="${joint['xyz']}"/>
+        <limit effort="${joint['effort']}" lower="${joint['lower']}" upper="${joint['upper']}" velocity="${joint['velocity']}"/>
+        <axis xyz="${joint['axis']}" />
+        <parent link="${links[n]['name']}" />
+        <child link="${links[n+1]['name']}" />
     </joint>
   </xacro:macro>
-  <!-- world link and joint-->
+  <!-- world link & world link to base link joint-->
   <link name="world" />
-  <joint name="world_to_${link_names[0]}" type="fixed">
+  <joint name="world_to_${links[0]['name']}" type="fixed">
     <origin rpy="0 0 0" xyz="0 0 0" />
     <parent link="world"/>
-    <child link="${link_names[0]}"/>
+    <child link="${links[0]['name']}"/>
   </joint>
   <!-- robot links and joints -->
-  <xacro:link number="0" />
-  <xacro:joint number="0" lower="${-3 * PI / 2}" upper="${3 * PI / 2}" velocity="0.5" axis="0 0 1" />
-  <xacro:link number="1" />
-  <xacro:joint number="1" lower="${-1 * PI / 2}" upper="${PI / 2}" velocity="0.5" axis="1 0 0" />
-  <xacro:link number="2" />
-  <xacro:joint number="2" lower="${-1 * PI / 3}" upper="${PI / 2}" velocity="0.5" axis="1 0 0" />
-  <xacro:link number="3" />
+  <xacro:link link="${links[0]}" />
+  <xacro:joint joint="${joints[0]}" n="0" />
+  <xacro:link link="${links[1]}" />
+  <xacro:joint joint="${joints[1]}" n="1" />
+  <xacro:link link="${links[2]}" />
+  <xacro:joint joint="${joints[2]}" n="2" />
+  <xacro:link link="${links[3]}" />
+  <xacro:joint joint="${joints[3]}" n="3" />
+  <xacro:link link="${links[4]}" />
 </robot>

Commit message: test

File: rpd_robot_description/urdf/rpd_robot.urdf.xacro (robot description, xacro)
@@ -1,6 +1,20 @@
 <?xml version="1.0"?>
 <robot name="rpd_robot" xmlns:xacro="http://www.ros.org/wiki/xacro">
+  <xacro:arg name="port" default="/dev/ttyACM0" />
+  <xacro:arg name="baudrate" default="115200" />
+  <xacro:arg name="use_sim" default="false" />
+  <xacro:arg name="use_mock_hardware" default="false" />
+  <xacro:arg name="mock_sensor_commands" default="false" />
   <material name="black">
     <color rgba="0 0 0 1"/>
+  </material>
+  <material name="red">
+    <color rgba="1 0 0 1"/>
+  </material>
+  <material name="green">
+    <color rgba="0 1 0 1"/>
+  </material>
+  <material name="blue">
+    <color rgba="0 0 1 1"/>
   </material>
   <xacro:property name="description_pkg" value="$(find rpd_robot_description)" />
@@ -10,6 +24,5 @@
   <xacro:property name="joints" value="${config['joints']}" />
   <xacro:include filename="${description_pkg}/urdf/rpd_robot_arm.urdf.xacro"/>
-  <xacro:include filename="${description_pkg}/urdf/rpd_robot_gripper.urdf.xacro"/>
+  <xacro:include filename="${description_pkg}/urdf/rpd_robot_gazebo.xacro"/>
   <xacro:include filename="${description_pkg}/urdf/rpd_robot_ros2_control.xacro"/>
-  <!-- <xacro:include filename="${description_pkg}/urdf/rpd_robot_gazebo.xacro"/> -->
 </robot>

File: rpd_robot_description/urdf/rpd_robot_arm.urdf.xacro (robot description, xacro)
@@ -5,5 +5,5 @@
     <origin rpy="0 0 0" xyz="${link['xyz']}" />
     <geometry>
-      <mesh filename="file://${description_pkg}/meshes/${link['name']}.stl" />
+      <mesh filename="file://${description_pkg}/meshes/${link['name']}.stl" /> <!-- package -->
     </geometry>
   </xacro:macro>
@@ -22,21 +22,26 @@
     <link name="${link['name']}">
         <visual>
-        <xacro:origin_geometry link="${link}" />
-        <material name="${link['color']}" />
+          <xacro:origin_geometry link="${link}" />
+          <material name="${link['color']}" />
         </visual>
         <collision>
-        <xacro:origin_geometry link="${link}" />
+          <xacro:origin_geometry link="${link}" /> <!-- box geo -->
         </collision>
-        <!-- <xacro:inertial n="${links[n]}" /> -->
+        <xacro:inertial link="${link}" />
     </link>
   </xacro:macro>
  <!-- joint macro -->
-  <xacro:macro name="joint" params="joint n">
-    <joint name="${joint['name']}" type="revolute"> <!-- can keep continuous for joint_1 -->
-        <origin rpy="0 0 0" xyz="${joint['xyz']}"/>
-        <limit effort="${joint['effort']}" lower="${joint['lower']}" upper="${joint['upper']}" velocity="${joint['velocity']}"/>
+  <xacro:macro name="joint" params="joint is_fixed:=false">
+    <joint name="${joint['name']}" type="${joint['type']}">
+      <origin rpy="0 0 0" xyz="${joint['xyz']}" />
+      <xacro:if value="${not is_fixed}">
+        <limit effort="${joint['effort']}" lower="${joint['lower']}" upper="${joint['upper']}" velocity="${joint['velocity']}" />
         <axis xyz="${joint['axis']}" />
-        <parent link="${links[n]['name']}" />
-        <child link="${links[n+1]['name']}" />
+      </xacro:if>
+        <parent link="${joint['parent']}" />
+        <child link="${joint['child']}" />
+      <xacro:if value="${joint['mimic']['use']}">
+        <mimic joint="${joint['mimic']['joint']}" multiplier="${joint['mimic']['multiplier']}" />
+      </xacro:if>
     </joint>
   </xacro:macro>
@@ -50,11 +55,26 @@
   <!-- robot links and joints -->
   <xacro:link link="${links[0]}" />
-  <xacro:joint joint="${joints[0]}" n="0" />
+  <xacro:joint joint="${joints[0]}" />
   <xacro:link link="${links[1]}" />
-  <xacro:joint joint="${joints[1]}" n="1" />
+  <xacro:joint joint="${joints[1]}" />
   <xacro:link link="${links[2]}" />
-  <xacro:joint joint="${joints[2]}" n="2" />
+  <xacro:joint joint="${joints[2]}" />
   <xacro:link link="${links[3]}" />
-  <xacro:joint joint="${joints[3]}" n="3" />
+  <xacro:joint joint="${joints[3]}" />
   <xacro:link link="${links[4]}" />
+  <xacro:joint joint="${joints[4]}" />
+  <xacro:link link="${links[5]}" />
+  <xacro:joint joint="${joints[5]}" />
+  <xacro:link link="${links[6]}" />
+  <!-- end effector link and joint -->
+  <xacro:joint joint="${joints[6]}" is_fixed="true" />
+  <link name="${links[7]['name']}">
+    <visual>
+      <origin rpy="0 0 0" xyz="${links[7]['xyz']}" />
+      <geometry>
+        <box size="${links[7]['size']}" />
+      </geometry>
+      <material name="${links[7]['color']}"/>
+    </visual>
+  </link>
 </robot>

File: rpd_robot_description/urdf/rpd_robot_gazebo.xacro (robot description, xacro)
@@ -11,20 +11,27 @@
     </gazebo>
   </xacro:macro>
+  <xacro:gz_link_physical_properties reference="base_link"/>
   <xacro:gz_link_physical_properties reference="link_1"/>
   <xacro:gz_link_physical_properties reference="link_2"/>
   <xacro:gz_link_physical_properties reference="link_3"/>
-  <!-- <xacro:Link reference="link_4"/> -->
+  <xacro:gz_link_physical_properties reference="gripper_link"/>
   <xacro:gz_link_physical_properties reference="gripper_left_link"/>
   <xacro:gz_link_physical_properties reference="gripper_right_link"/>
-  <gazebo reference="gripper_link" />
+  <gazebo reference="ee_link" />
 <gazebo>
-    <plugin filename="" name="" />
-</gazebo>
-<gazebo>
-    <plugin filename="gz-sim-joint-state-publisher" name="gz::sim::systems::JointStatePublisher">
+    <plugin filename="gz-sim-joint-state-publisher-system" name="gz::sim::systems::JointStatePublisher">
+      <joint_name>world_to_${links[0]['name']}</joint_name>
       <joint_name>joint_1</joint_name>
       <joint_name>joint_2</joint_name>
       <joint_name>joint_3</joint_name>
+      <joint_name>joint_4</joint_name>
+      <joint_name>gripper_left_joint</joint_name>
+      <joint_name>gripper_right_joint</joint_name>
     </plugin>
 </gazebo>
+  <gazebo>
+    <plugin filename="gz_ros2_control-system" name="gz_ros2_control::GazeboSimROS2ControlPlugin">
+      <parameters>$(find rpd_robot_bringup)/config/rpd_robot_controllers.yaml</parameters>
+    </plugin>
+  </gazebo>
 </robot>

File: rpd_robot_description/urdf/rpd_robot_ros2_control.xacro (robot description, xacro)
@@ -3,19 +3,45 @@
   <ros2_control name="RoboparadigmRobotSystem" type="system">
     <hardware>
-      <plugin>mock_components/GenericSystem</plugin>
-      <param name="state_following_offset">0.0</param>
-      <param name="calculate_dynamics">true</param>
+      <xacro:if value="$(arg use_sim)">
+        <plugin>gz_ros2_control/GazeboSimSystem</plugin>
+      </xacro:if>
+      <xacro:unless value="$(arg use_sim)">
+        <xacro:if value="$(arg use_mock_hardware)">
+          <plugin>mock_components/GenericSystem</plugin>
+          <!-- <param name="mock_sensor_commands">$(arg mock_sensor_commands)</param> -->
+          <param name="state_following_offset">0.0</param>
+        </xacro:if>
+        <xacro:unless value="$(arg use_mock_hardware)">
+          <plugin>rpd_robot_hardware/RpdRobotHardwareInterface</plugin>
+          <param name="port">$(arg port)</param>
+          <param name="baudrate">$(arg baudrate)</param>
+        </xacro:unless>
+      </xacro:unless>
     </hardware>
-    <xacro:macro name="joint_control" params="n">
-      <joint name="${joints[n]['name']}">
-          <command_interface name="position"/>
-          <state_interface name="position"/>
-          <state_interface name="velocity"/>
-          <state_interface name="effort"/>
+    <xacro:macro name="joint_control" params="joint">
+      <joint name="${joint['name']}">
+        <param name="motor_id">${joint['motor_id']}</param>
+        <command_interface name="position"/>
+        <command_interface name="velocity"/>
+        <command_interface name="acceleration"/>
+        <state_interface name="position"/>
+        <state_interface name="velocity"/>
+        <state_interface name="acceleration"/>
       </joint>
     </xacro:macro>
-    <xacro:joint_control n="0" />
-    <xacro:joint_control n="1" />
-    <xacro:joint_control n="2" />
+    <xacro:joint_control joint="${joints[0]}" />
+    <xacro:joint_control joint="${joints[1]}" />
+    <xacro:joint_control joint="${joints[2]}" />
+    <xacro:joint_control joint="${joints[3]}" />
+    <xacro:joint_control joint="${joints[4]}" />
+    <xacro:if value="$(arg use_sim)">
+      <joint name="${joints[5]['name']}">
+        <param name="mimic">${joints[5]['mimic']['joint']}</param>
+        <param name="multiplier">${joints[5]['mimic']['multiplier']}</param>
+        <state_interface name="position"/>
+        <state_interface name="velocity"/>
+        <state_interface name="acceleration"/>
+      </joint>
+    </xacro:if>
   </ros2_control>
 </robot>

Commit message: test

File: rpd_robot_description/urdf/rpd_robot.urdf.xacro (robot description, xacro)
@@ -2,8 +2,7 @@
 <robot name="rpd_robot" xmlns:xacro="http://www.ros.org/wiki/xacro">
   <xacro:arg name="port" default="/dev/ttyACM0" />
-  <xacro:arg name="baudrate" default="115200" />
+  <xacro:arg name="baudrate" default="1000000" />
   <xacro:arg name="use_sim" default="false" />
   <xacro:arg name="use_mock_hardware" default="false" />
-  <xacro:arg name="mock_sensor_commands" default="false" />
   <material name="black">
     <color rgba="0 0 0 1"/>

File: rpd_robot_description/urdf/rpd_robot_arm.urdf.xacro (robot description, xacro)
@@ -1,14 +1,21 @@
 <?xml version="1.0"?>
 <robot xmlns:xacro="http://www.ros.org/wiki/xacro">
-  <!-- origin and geometry macro -->
-  <xacro:macro name="origin_geometry" params="link">
-    <origin rpy="0 0 0" xyz="${link['xyz']}" />
-    <geometry>
-      <mesh filename="file://${description_pkg}/meshes/${link['name']}.stl" /> <!-- package -->
-    </geometry>
-  </xacro:macro>
-  <!-- Inertial macro -->
-  <xacro:macro name="inertial" params="link">
-    <inertial>
+  <!-- link macro -->
+  <xacro:macro name="link" params="link color:=black">
+    <link name="${link['name']}">
+        <visual>
+          <origin rpy="0 0 0" xyz="${link['xyz']}" />
+          <geometry>
+            <mesh filename="file://${description_pkg}/meshes/${link['name']}.stl" />
+          </geometry>
+          <material name="${link['color']}" />
+        </visual>
+        <collision>
+          <origin rpy="0 0 0" xyz="${link['xyz']}" />
+          <geometry>
+            <mesh filename="file://${description_pkg}/meshes/${link['name']}.stl" />  <!-- box geo -->
+          </geometry>
+        </collision>
+        <inertial>
       <mass value="${link['mass']}" />
       <origin xyz="${link['com']}" rpy="0 0 0"/>
@@ -17,28 +24,14 @@
                izz="${link['inertia']['izz']}" />
     </inertial>
-  </xacro:macro>
-  <!-- link macro -->
-  <xacro:macro name="link" params="link color:=black">
-    <link name="${link['name']}">
-        <visual>
-          <xacro:origin_geometry link="${link}" />
-          <material name="${link['color']}" />
-        </visual>
-        <collision>
-          <xacro:origin_geometry link="${link}" /> <!-- box geo -->
-        </collision>
-        <xacro:inertial link="${link}" />
     </link>
   </xacro:macro>
  <!-- joint macro -->
-  <xacro:macro name="joint" params="joint is_fixed:=false">
+  <xacro:macro name="joint" params="joint">
     <joint name="${joint['name']}" type="${joint['type']}">
       <origin rpy="0 0 0" xyz="${joint['xyz']}" />
-      <xacro:if value="${not is_fixed}">
-        <limit effort="${joint['effort']}" lower="${joint['lower']}" upper="${joint['upper']}" velocity="${joint['velocity']}" />
-        <axis xyz="${joint['axis']}" />
-      </xacro:if>
-        <parent link="${joint['parent']}" />
-        <child link="${joint['child']}" />
+      <limit effort="${joint['effort']}" lower="${joint['lower']}" upper="${joint['upper']}" velocity="${joint['velocity']}" />
+      <axis xyz="${joint['axis']}" />
+      <parent link="${joint['parent']}" />
+      <child link="${joint['child']}" />
       <xacro:if value="${joint['mimic']['use']}">
         <mimic joint="${joint['mimic']['joint']}" multiplier="${joint['mimic']['multiplier']}" />
@@ -68,5 +61,9 @@
   <xacro:link link="${links[6]}" />
   <!-- end effector link and joint -->
-  <xacro:joint joint="${joints[6]}" is_fixed="true" />
+  <joint name="${joints[6]['name']}" type="fixed">
+    <origin rpy="0 0 0" xyz="${joints[6]['xyz']}" />
+    <parent link="${joints[6]['parent']}" />
+    <child link="${joints[6]['child']}" />
+  </joint>
   <link name="${links[7]['name']}">
     <visual>

File: rpd_robot_description/urdf/rpd_robot_gazebo.xacro (robot description, xacro)
@@ -22,10 +22,10 @@
     <plugin filename="gz-sim-joint-state-publisher-system" name="gz::sim::systems::JointStatePublisher">
       <joint_name>world_to_${links[0]['name']}</joint_name>
-      <joint_name>joint_1</joint_name>
-      <joint_name>joint_2</joint_name>
-      <joint_name>joint_3</joint_name>
-      <joint_name>joint_4</joint_name>
-      <joint_name>gripper_left_joint</joint_name>
-      <joint_name>gripper_right_joint</joint_name>
+      <joint_name>${joints[0]['name']}</joint_name>
+      <joint_name>${joints[1]['name']}</joint_name>
+      <joint_name>${joints[2]['name']}</joint_name>
+      <joint_name>${joints[3]['name']}</joint_name>
+      <joint_name>${joints[4]['name']}</joint_name>
+      <joint_name>${joints[5]['name']}</joint_name>
     </plugin>
 </gazebo>

File: rpd_robot_description/urdf/rpd_robot_ros2_control.xacro (robot description, xacro)
@@ -9,5 +9,4 @@
         <xacro:if value="$(arg use_mock_hardware)">
           <plugin>mock_components/GenericSystem</plugin>
-          <!-- <param name="mock_sensor_commands">$(arg mock_sensor_commands)</param> -->
           <param name="state_following_offset">0.0</param>
         </xacro:if>
@@ -23,9 +22,9 @@
         <param name="motor_id">${joint['motor_id']}</param>
         <command_interface name="position"/>
-        <command_interface name="velocity"/>
-        <command_interface name="acceleration"/>
+        <!-- <command_interface name="velocity"/> -->
+        <!-- <command_interface name="acceleration"/> -->
         <state_interface name="position"/>
         <state_interface name="velocity"/>
-        <state_interface name="acceleration"/>
+        <!-- <state_interface name="acceleration"/> -->
       </joint>
     </xacro:macro>
@@ -41,5 +40,5 @@
         <state_interface name="position"/>
         <state_interface name="velocity"/>
-        <state_interface name="acceleration"/>
+        <!-- <state_interface name="acceleration"/> -->
       </joint>
     </xacro:if>
